Commit message: Add iCub3 right leg urdf

File: matlab/urdf/iCub3_right_leg.urdf (robot description, URDF)
Before this commit: robot iDynTreeURDFModelExportModelName, 214 links, 213 joints
Links:
- removed link chest_ems_acc_eb1
- removed link chest_ems_acc_eb2
- removed link chest_ems_acc_eb3
- removed link chest_ems_acc_eb4
- removed link chest_ems_gyro_eb1
- removed link chest_ems_gyro_eb2
- removed link chest_ems_gyro_eb3
- removed link chest_ems_gyro_eb4
- removed link chest_mtb_acc_0b10
- removed link chest_mtb_acc_0b7
- removed link chest_mtb_acc_0b8
- removed link chest_mtb_acc_0b9
- removed link head_imu_acc_1x1
- removed link imu_frame
- removed link l_foot
- removed link l_foot_dh_frame
- removed link l_foot_ft_sensor
- removed link l_foot_mtb_acc_10b12
- removed link l_foot_mtb_acc_10b13
- removed link l_forearm_dh_frame
- removed link l_forearm_mtb_acc_1b7
- removed link l_forearm_mtb_acc_1b8
- removed link l_forearm_mtb_acc_1b9
- removed link l_forearm_skin_0
- removed link l_forearm_skin_1
- removed link l_forearm_skin_10
- removed link l_forearm_skin_11
- removed link l_forearm_skin_12
- removed link l_forearm_skin_13
- removed link l_forearm_skin_14
- removed link l_forearm_skin_15
- removed link l_forearm_skin_16
- removed link l_forearm_skin_17
- removed link l_forearm_skin_19
- removed link l_forearm_skin_2
- removed link l_forearm_skin_22
- removed link l_forearm_skin_24
- removed link l_forearm_skin_25
- removed link l_forearm_skin_28
- removed link l_forearm_skin_29
- removed link l_forearm_skin_3
- removed link l_forearm_skin_4
- removed link l_forearm_skin_5
- removed link l_forearm_skin_6
- removed link l_forearm_skin_7
- removed link l_forearm_skin_8
- removed link l_forearm_skin_9
- removed link l_hand_dh_frame
- removed link l_lower_leg_ems_acc_eb7
- removed link l_lower_leg_ems_gyro_eb7
- removed link l_lower_leg_mtb_acc_10b10
- removed link l_lower_leg_mtb_acc_10b11
- removed link l_lower_leg_mtb_acc_10b8
- removed link l_lower_leg_mtb_acc_10b9
- removed link l_upper_arm_mtb_acc_1b10
- removed link l_upper_arm_mtb_acc_1b11
- removed link l_upper_arm_mtb_acc_1b12
- removed link l_upper_arm_mtb_acc_1b13
- removed link l_upper_leg_back_contact
- removed link l_upper_leg_dh_frame
- removed link l_upper_leg_ems_acc_eb10
- removed link l_upper_leg_ems_acc_eb6
- removed link l_upper_leg_ems_gyro_eb10
- removed link l_upper_leg_ems_gyro_eb6
- removed link l_upper_leg_mtb_acc_10b1
- removed link l_upper_leg_mtb_acc_10b2
- removed link l_upper_leg_mtb_acc_10b3
- removed link l_upper_leg_mtb_acc_10b4
- removed link l_upper_leg_mtb_acc_10b5
- removed link l_upper_leg_mtb_acc_10b6
- removed link l_upper_leg_mtb_acc_10b7
- removed link r_foot
- removed link r_foot_dh_frame
- removed link r_foot_ft_sensor
- removed link r_foot_mtb_acc_11b12
- removed link r_foot_mtb_acc_11b13
- removed link r_forearm_dh_frame
- removed link r_forearm_mtb_acc_2b7
- removed link r_forearm_mtb_acc_2b8
- removed link r_forearm_mtb_acc_2b9
- removed link r_forearm_skin_0
- removed link r_forearm_skin_1
- removed link r_forearm_skin_10
- removed link r_forearm_skin_11
- removed link r_forearm_skin_12
- removed link r_forearm_skin_13
- removed link r_forearm_skin_14
- removed link r_forearm_skin_15
- removed link r_forearm_skin_16
- removed link r_forearm_skin_17
- removed link r_forearm_skin_19
- removed link r_forearm_skin_2
- removed link r_forearm_skin_22
- removed link r_forearm_skin_24
- removed link r_forearm_skin_25
- removed link r_forearm_skin_28
- removed link r_forearm_skin_29
- removed link r_forearm_skin_3
- removed link r_forearm_skin_4
- removed link r_forearm_skin_5
- removed link r_forearm_skin_6
- removed link r_forearm_skin_7
- removed link r_forearm_skin_8
- removed link r_forearm_skin_9
- removed link r_hand_dh_frame
- removed link r_lower_leg_ems_acc_eb9
- removed link r_lower_leg_ems_gyro_eb9
- removed link r_lower_leg_mtb_acc_11b10
- removed link r_lower_leg_mtb_acc_11b11
- removed link r_lower_leg_mtb_acc_11b8
- removed link r_lower_leg_mtb_acc_11b9
- removed link r_lower_leg_skin_0
- removed link r_lower_leg_skin_10
- removed link r_lower_leg_skin_11
- removed link r_lower_leg_skin_14
- removed link r_lower_leg_skin_15
- removed link r_lower_leg_skin_16
- removed link r_lower_leg_skin_17
- removed link r_lower_leg_skin_19
- removed link r_lower_leg_skin_20
- removed link r_lower_leg_skin_21
- removed link r_lower_leg_skin_28
- removed link r_lower_leg_skin_29
- removed link r_lower_leg_skin_3
- removed link r_lower_leg_skin_31
- removed link r_lower_leg_skin_32
- removed link r_lower_leg_skin_35
- removed link r_lower_leg_skin_36
- removed link r_lower_leg_skin_37
- removed link r_lower_leg_skin_38
- removed link r_lower_leg_skin_4
- removed link r_lower_leg_skin_41
- removed link r_lower_leg_skin_42
- removed link r_lower_leg_skin_43
- removed link r_lower_leg_skin_46
- removed link r_lower_leg_skin_47
- removed link r_lower_leg_skin_49
- removed link r_lower_leg_skin_5
- removed link r_lower_leg_skin_50
- removed link r_lower_leg_skin_51
- removed link r_lower_leg_skin_52
- removed link r_lower_leg_skin_53
- removed link r_lower_leg_skin_54
- removed link r_lower_leg_skin_55
- removed link r_lower_leg_skin_56
- removed link r_lower_leg_skin_6
- removed link r_lower_leg_skin_60
- removed link r_lower_leg_skin_61
- removed link r_lower_leg_skin_9
- removed link r_upper_arm_mtb_acc_2b10
- removed link r_upper_arm_mtb_acc_2b11
- removed link r_upper_arm_mtb_acc_2b12
- removed link r_upper_arm_mtb_acc_2b13
- removed link r_upper_leg_back_contact
- removed link r_upper_leg_dh_frame
- removed link r_upper_leg_ems_acc_eb11
- removed link r_upper_leg_ems_acc_eb8
- removed link r_upper_leg_ems_gyro_eb11
- removed link r_upper_leg_ems_gyro_eb8
- removed link r_upper_leg_mtb_acc_11b1
- removed link r_upper_leg_mtb_acc_11b2
- removed link r_upper_leg_mtb_acc_11b3
- removed link r_upper_leg_mtb_acc_11b4
- removed link r_upper_leg_mtb_acc_11b5
- removed link r_upper_leg_mtb_acc_11b6
- removed link r_upper_leg_mtb_acc_11b7
- removed link root_link_ems_acc_eb5
- removed link root_link_ems_gyro_eb5
- removed link root_link_imu_acc
- removed link root_link_imu_frame
- added link l_foot_front
- added link l_foot_front_ft_sensor
- added link l_foot_rear
- added link l_foot_rear_ft_sensor
- added link neck_3
- added link r_foot_front
- added link r_foot_front_ft_sensor
- added link r_foot_rear
- added link r_foot_rear_ft_sensor
- link r_ankle_1: mass 0.6803 -> 1.80595; geometry collision mesh filename=package://iCub/meshes/simmechanics/sim_icub3_r_ankle_1_prt.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 scale=0.001 0.001 0.001; visual mesh filename=package://iCub/meshes/simmechanics/sim_icub3_r_ankle_1_prt.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 scale=0.001 0.001 0.001
- link r_ankle_2: mass 0.623218 -> 1.43897637; geometry collision mesh filename=package://iCub/meshes/simmechanics/sim_icub3_r_ankle_2_prt.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 scale=0.001 0.001 0.001; collision mesh filename=package://iCub/meshes/simmechanics/sim_icub3_r_foot_front_p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 scale=0.001 0.001 0.001
- link r_hip_1: mass 0.919978 -> 2.48546; geometry collision mesh filename=package://iCub/meshes/simmechanics/sim_icub3_r_hip_1_prt.stl scale=0.001 0.001 0.001; visual mesh filename=package://iCub/meshes/simmechanics/sim_icub3_r_hip_1_prt.stl scale=0.001 0.001 0.001
- link r_hip_2: mass 0.544573 -> 4.17692; geometry collision mesh filename=package://iCub/meshes/simmechanics/sim_icub3_r_hip_2_prt.stl scale=0.001 0.001 0.001; collision mesh filename=package://iCub/meshes/simmechanics/sim_icub3_r_hip_3_prt.stl scale=0.001 0.001 0.001
- link r_lower_leg: mass 1.472 -> 4.59072; geometry collision mesh filename=package://iCub/meshes/simmechanics/sim_icub3_r_lower_leg_pr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 scale=0.001 0.001 0.001; visual mesh filename=package://iCub/meshes/simmechanics/sim_icub3_r_lower_leg_pr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 scale=0.001 0.001 0.001
- link r_upper_leg: mass 1.8035 -> 2.24396; geometry collision mesh filename=package://iCub/meshes/simmechanics/sim_icub3_r_upper_leg_pr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 scale=0.001 0.001 0.001; visual mesh filename=package://iCub/meshes/simmechanics/sim_icub3_r_upper_leg_pr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 scale=0.001 0.001 0.001
- link root_link: mass 27.0146597 -> 42.30274274; geometry collision mesh filename=package://iCub/meshes/simmechanics/sim_icub3_chest_prt.stl scale=0.001 0.001 0.001; collision mesh filename=package://iCub/meshes/simmechanics/sim_icub3_head_prt.stl scale=0.001 0.001 0.001
Joints:
- removed joint chest_ems_acc_eb1_fixed_joint
- removed joint chest_ems_acc_eb2_fixed_joint
- removed joint chest_ems_acc_eb3_fixed_joint
- removed joint chest_ems_acc_eb4_fixed_joint
- removed joint chest_ems_gyro_eb1_fixed_joint
- removed joint chest_ems_gyro_eb2_fixed_joint
- removed joint chest_ems_gyro_eb3_fixed_joint
- removed joint chest_ems_gyro_eb4_fixed_joint
- removed joint chest_mtb_acc_0b10_fixed_joint
- removed joint chest_mtb_acc_0b7_fixed_joint
- removed joint chest_mtb_acc_0b8_fixed_joint
- removed joint chest_mtb_acc_0b9_fixed_joint
- removed joint head_imu_acc_1x1_fixed_joint
- removed joint imu_frame_fixed_joint
- removed joint l_foot_dh_frame_fixed_joint
- removed joint l_foot_fixed_joint
- removed joint l_foot_ft_sensor_fixed_joint
- removed joint l_foot_mtb_acc_10b12_fixed_joint
- removed joint l_foot_mtb_acc_10b13_fixed_joint
- removed joint l_forearm_dh_frame_fixed_joint
- removed joint l_forearm_mtb_acc_1b7_fixed_joint
- removed joint l_forearm_mtb_acc_1b8_fixed_joint
- removed joint l_forearm_mtb_acc_1b9_fixed_joint
- removed joint l_forearm_skin_0_fixed_joint
- removed joint l_forearm_skin_10_fixed_joint
- removed joint l_forearm_skin_11_fixed_joint
- removed joint l_forearm_skin_12_fixed_joint
- removed joint l_forearm_skin_13_fixed_joint
- removed joint l_forearm_skin_14_fixed_joint
- removed joint l_forearm_skin_15_fixed_joint
- removed joint l_forearm_skin_16_fixed_joint
- removed joint l_forearm_skin_17_fixed_joint
- removed joint l_forearm_skin_19_fixed_joint
- removed joint l_forearm_skin_1_fixed_joint
- removed joint l_forearm_skin_22_fixed_joint
- removed joint l_forearm_skin_24_fixed_joint
- removed joint l_forearm_skin_25_fixed_joint
- removed joint l_forearm_skin_28_fixed_joint
- removed joint l_forearm_skin_29_fixed_joint
- removed joint l_forearm_skin_2_fixed_joint
- removed joint l_forearm_skin_3_fixed_joint
- removed joint l_forearm_skin_4_fixed_joint
- removed joint l_forearm_skin_5_fixed_joint
- removed joint l_forearm_skin_6_fixed_joint
- removed joint l_forearm_skin_7_fixed_joint
- removed joint l_forearm_skin_8_fixed_joint
- removed joint l_forearm_skin_9_fixed_joint
- removed joint l_hand_dh_frame_fixed_joint
- removed joint l_lower_leg_ems_acc_eb7_fixed_joint
- removed joint l_lower_leg_ems_gyro_eb7_fixed_joint
- removed joint l_lower_leg_mtb_acc_10b10_fixed_joint
- removed joint l_lower_leg_mtb_acc_10b11_fixed_joint
- removed joint l_lower_leg_mtb_acc_10b8_fixed_joint
- removed joint l_lower_leg_mtb_acc_10b9_fixed_joint
- removed joint l_upper_arm_mtb_acc_1b10_fixed_joint
- removed joint l_upper_arm_mtb_acc_1b11_fixed_joint
- removed joint l_upper_arm_mtb_acc_1b12_fixed_joint
- removed joint l_upper_arm_mtb_acc_1b13_fixed_joint
- removed joint l_upper_leg_back_contact_fixed_joint
- removed joint l_upper_leg_dh_frame_fixed_joint
- removed joint l_upper_leg_ems_acc_eb10_fixed_joint
- removed joint l_upper_leg_ems_acc_eb6_fixed_joint
- removed joint l_upper_leg_ems_gyro_eb10_fixed_joint
- removed joint l_upper_leg_ems_gyro_eb6_fixed_joint
- removed joint l_upper_leg_mtb_acc_10b1_fixed_joint
- removed joint l_upper_leg_mtb_acc_10b2_fixed_joint
- removed joint l_upper_leg_mtb_acc_10b3_fixed_joint
- removed joint l_upper_leg_mtb_acc_10b4_fixed_joint
- removed joint l_upper_leg_mtb_acc_10b5_fixed_joint
- removed joint l_upper_leg_mtb_acc_10b6_fixed_joint
- removed joint l_upper_leg_mtb_acc_10b7_fixed_joint
- removed joint r_foot_dh_frame_fixed_joint
- removed joint r_foot_fixed_joint
- removed joint r_foot_ft_sensor_fixed_joint
- removed joint r_foot_mtb_acc_11b12_fixed_joint
- removed joint r_foot_mtb_acc_11b13_fixed_joint
- removed joint r_forearm_dh_frame_fixed_joint
- removed joint r_forearm_mtb_acc_2b7_fixed_joint
- removed joint r_forearm_mtb_acc_2b8_fixed_joint
- removed joint r_forearm_mtb_acc_2b9_fixed_joint
- removed joint r_forearm_skin_0_fixed_joint
- removed joint r_forearm_skin_10_fixed_joint
- removed joint r_forearm_skin_11_fixed_joint
- removed joint r_forearm_skin_12_fixed_joint
- removed joint r_forearm_skin_13_fixed_joint
- removed joint r_forearm_skin_14_fixed_joint
- removed joint r_forearm_skin_15_fixed_joint
- removed joint r_forearm_skin_16_fixed_joint
- removed joint r_forearm_skin_17_fixed_joint
- removed joint r_forearm_skin_19_fixed_joint
- removed joint r_forearm_skin_1_fixed_joint
- removed joint r_forearm_skin_22_fixed_joint
- removed joint r_forearm_skin_24_fixed_joint
- removed joint r_forearm_skin_25_fixed_joint
- removed joint r_forearm_skin_28_fixed_joint
- removed joint r_forearm_skin_29_fixed_joint
- removed joint r_forearm_skin_2_fixed_joint
- removed joint r_forearm_skin_3_fixed_joint
- removed joint r_forearm_skin_4_fixed_joint
- removed joint r_forearm_skin_5_fixed_joint
- removed joint r_forearm_skin_6_fixed_joint
- removed joint r_forearm_skin_7_fixed_joint
- removed joint r_forearm_skin_8_fixed_joint
- removed joint r_forearm_skin_9_fixed_joint
- removed joint r_hand_dh_frame_fixed_joint
- removed joint r_lower_leg_ems_acc_eb9_fixed_joint
- removed joint r_lower_leg_ems_gyro_eb9_fixed_joint
- removed joint r_lower_leg_mtb_acc_11b10_fixed_joint
- removed joint r_lower_leg_mtb_acc_11b11_fixed_joint
- removed joint r_lower_leg_mtb_acc_11b8_fixed_joint
- removed joint r_lower_leg_mtb_acc_11b9_fixed_joint
- removed joint r_lower_leg_skin_0_fixed_joint
- removed joint r_lower_leg_skin_10_fixed_joint
- removed joint r_lower_leg_skin_11_fixed_joint
- removed joint r_lower_leg_skin_14_fixed_joint
- removed joint r_lower_leg_skin_15_fixed_joint
- removed joint r_lower_leg_skin_16_fixed_joint
- removed joint r_lower_leg_skin_17_fixed_joint
- removed joint r_lower_leg_skin_19_fixed_joint
- removed joint r_lower_leg_skin_20_fixed_joint
- removed joint r_lower_leg_skin_21_fixed_joint
- removed joint r_lower_leg_skin_28_fixed_joint
- removed joint r_lower_leg_skin_29_fixed_joint
- removed joint r_lower_leg_skin_31_fixed_joint
- removed joint r_lower_leg_skin_32_fixed_joint
- removed joint r_lower_leg_skin_35_fixed_joint
- removed joint r_lower_leg_skin_36_fixed_joint
- removed joint r_lower_leg_skin_37_fixed_joint
- removed joint r_lower_leg_skin_38_fixed_joint
- removed joint r_lower_leg_skin_3_fixed_joint
- removed joint r_lower_leg_skin_41_fixed_joint
- removed joint r_lower_leg_skin_42_fixed_joint
- removed joint r_lower_leg_skin_43_fixed_joint
- removed joint r_lower_leg_skin_46_fixed_joint
- removed joint r_lower_leg_skin_47_fixed_joint
- removed joint r_lower_leg_skin_49_fixed_joint
- removed joint r_lower_leg_skin_4_fixed_joint
- removed joint r_lower_leg_skin_50_fixed_joint
- removed joint r_lower_leg_skin_51_fixed_joint
- removed joint r_lower_leg_skin_52_fixed_joint
- removed joint r_lower_leg_skin_53_fixed_joint
- removed joint r_lower_leg_skin_54_fixed_joint
- removed joint r_lower_leg_skin_55_fixed_joint
- removed joint r_lower_leg_skin_56_fixed_joint
- removed joint r_lower_leg_skin_5_fixed_joint
- removed joint r_lower_leg_skin_60_fixed_joint
- removed joint r_lower_leg_skin_61_fixed_joint
- removed joint r_lower_leg_skin_6_fixed_joint
- removed joint r_lower_leg_skin_9_fixed_joint
- removed joint r_upper_arm_mtb_acc_2b10_fixed_joint
- removed joint r_upper_arm_mtb_acc_2b11_fixed_joint
- removed joint r_upper_arm_mtb_acc_2b12_fixed_joint
- removed joint r_upper_arm_mtb_acc_2b13_fixed_joint
- removed joint r_upper_leg_back_contact_fixed_joint
- removed joint r_upper_leg_dh_frame_fixed_joint
- removed joint r_upper_leg_ems_acc_eb11_fixed_joint
- removed joint r_upper_leg_ems_acc_eb8_fixed_joint
- removed joint r_upper_leg_ems_gyro_eb11_fixed_joint
- removed joint r_upper_leg_ems_gyro_eb8_fixed_joint
- removed joint r_upper_leg_mtb_acc_11b1_fixed_joint
- removed joint r_upper_leg_mtb_acc_11b2_fixed_joint
- removed joint r_upper_leg_mtb_acc_11b3_fixed_joint
- removed joint r_upper_leg_mtb_acc_11b4_fixed_joint
- removed joint r_upper_leg_mtb_acc_11b5_fixed_joint
- removed joint r_upper_leg_mtb_acc_11b6_fixed_joint
- removed joint r_upper_leg_mtb_acc_11b7_fixed_joint
- removed joint root_link_ems_acc_eb5_fixed_joint
- removed joint root_link_ems_gyro_eb5_fixed_joint
- removed joint root_link_imu_acc_fixed_joint
- removed joint root_link_imu_frame_fixed_joint
- added joint l_foot_front_fixed_joint: type fixed, parent root_link, child l_foot_front, origin xyz=0.10854999999999998 0.06475 -0.6325890000000001 rpy=0 -0 0
- added joint l_foot_front_ft_sensor_fixed_joint: type fixed, parent root_link, child l_foot_front_ft_sensor, origin xyz=0.10854999999999998 0.06475 -0.6325890000000001 rpy=0 -0 0
- added joint l_foot_rear_fixed_joint: type fixed, parent root_link, child l_foot_rear, origin xyz=-0.010700000000000008 0.06475 -0.6325890000000001 rpy=0 -0 0
- added joint l_foot_rear_ft_sensor_fixed_joint: type fixed, parent root_link, child l_foot_rear_ft_sensor, origin xyz=-0.010700000000000008 0.06475 -0.6325890000000001 rpy=0 -0 0
- added joint neck_3_fixed_joint: type fixed, parent root_link, child neck_3, origin xyz=0.0048615099999999994 0 0.42127000000000003 rpy=0 -0 0
- added joint r_foot_front_fixed_joint: type fixed, parent r_ankle_2, child r_foot_front, origin xyz=0.13525 0 -0.06579999999999997 rpy=0 -0 0
- added joint r_foot_front_ft_sensor_fixed_joint: type fixed, parent r_ankle_2, child r_foot_front_ft_sensor, origin xyz=0.13525 0 -0.06579999999999997 rpy=0 -0 0
- added joint r_foot_rear_fixed_joint: type fixed, parent r_ankle_2, child r_foot_rear, origin xyz=0.016 0 -0.06579999999999997 rpy=0 -0 0
- added joint r_foot_rear_ft_sensor_fixed_joint: type fixed, parent r_ankle_2, child r_foot_rear_ft_sensor, origin xyz=0.016 0 -0.06579999999999997 rpy=0 -0 0
- joint chest_fixed_joint: origin xyz=-0.005497499999999947 1.9073498977142145e-10 0.08200000000000002 rpy=1.5707963267948961 -0 -1.5707963267948961 -> xyz=0 0 0.19747000000000003 rpy=0 -0 0
- joint head_fixed_joint: origin xyz=-0.010809299999999869 1.9073498693475152e-10 0.241953 rpy=1.5707963267948961 -0 -1.5707963267948961 -> xyz=0.0048615099999999994 0 0.4904200000000001 rpy=0 -0 0
- joint l_ankle_1_fixed_joint: origin xyz=0.007309000000000008 -0.07010000000000001 -0.5549379999999999 rpy=0 0.2617991794798451 -3.141592653589793 -> xyz=0.026049999999999997 0.08295000000000001 -0.5317890000000001 rpy=0 -0 0
- joint l_ankle_2_fixed_joint: origin xyz=0.007309000000000008 -0.07010000000000001 -0.5549379999999999 rpy=0 0.2617991794798451 -3.141592653589793 -> xyz=-0.02670000000000001 0.06475 -0.5667890000000001 rpy=0 -0 0
- joint l_arm_ft_sensor_fixed_joint: origin xyz=-0.025619799999999887 -0.109391 0.09499999999999996 rpy=3.1415926535897922 -1.1657341758564144e-15 -3.1415926535897927 -> xyz=0.01160250023188351 0.14719399989874468 0.2765873999902195 rpy=0.0790794230156212 -0.052031613930206826 -0.27527862099575323
- joint l_elbow_1_fixed_joint: origin xyz=-0.02561980000000001 -0.07539109999999993 0.015740000000000018 rpy=-3.141592653589789 1.3089970069677406 4.372177745413122e-15 -> xyz=0.031246122657570638 0.15209302229214877 0.13144299586628905 rpy=0.0790794230156212 -0.052031613930206826 -0.27527862099575323
- joint l_forearm_fixed_joint: origin xyz=-0.010619800000000014 -0.10939099999999993 -0.020060000000000022 rpy=-3.141592653589789 1.3089970069677406 4.372177745413122e-15 -> xyz=0.021311022773212826 0.16151002194112832 0.07576799578628049 rpy=0.0790794230156212 -0.052031613930206826 -0.27527862099575323
- joint l_hand_fixed_joint: origin xyz=-0.010919800000000073 -0.08989809999999984 -0.12656000000000003 rpy=-3.141592653589789 1.3089970069677406 4.372177745413122e-15 -> xyz=0.027938017812163745 0.16329101706262705 -0.031628925986897 rpy=0.0790794230156212 -0.052031613930206826 -0.27527862099575323
- joint l_hip_1_fixed_joint: origin xyz=0.006451499999999999 -0.026000000000000023 -0.11991299999999999 rpy=0 -0 -3.141592653589793 -> xyz=0.0216 0.04045000000000001 0 rpy=0 -0 0
- joint l_hip_2_fixed_joint: origin xyz=0.006451500000000004 -0.07010000000000001 -0.11991299999999999 rpy=0 -0 -3.141592653589793 -> xyz=-0.02565 0.07355 -0.009000000000000008 rpy=0 -0 0
- joint l_hip_3_fixed_joint: origin xyz=0.007309000000000008 -0.07010000000000001 -0.19421299999999994 rpy=3.141592653589793 -0 -3.141592653589793 -> xyz=0.011049999999999997 0.07355 -0.09869999999999995 rpy=0 -0 0
- joint l_leg_ft_sensor_fixed_joint: origin xyz=0.007309000000000008 -0.07010000000000001 -0.19421299999999994 rpy=3.141592653589793 -0 -3.141592653589793 -> xyz=0.011049999999999997 0.07355 -0.09869999999999995 rpy=0 -0 0
- joint l_lower_leg_fixed_joint: origin xyz=0.007309000000000008 -0.07010000000000001 -0.3544379999999999 rpy=0 -0 -3.141592653589793 -> xyz=0.026049999999999997 0.08345000000000001 -0.2758 rpy=0 -0 0
- joint l_shoulder_1_fixed_joint: origin xyz=-0.013466799999999838 -0.12001600000000003 0.1748 rpy=1.5707963267948961 -0 -1.5707963267948961 -> xyz=-0.020835100000000002 0.0397423 0.3026729 rpy=0.2532616237670649 -1.1982921379466467e-7 -0.26179930185680106
- joint l_shoulder_2_fixed_joint: origin xyz=-0.021987199999999846 -0.10634500000000001 0.1748 rpy=-3.141592629949765 1.3089970275211211 -0.26179927643926154 -> xyz=0.011907900000000013 0.14265000000000003 0.3308707 rpy=0.0790794230156212 -0.052031613930206826 -0.27527862099575323
- joint l_shoulder_3_fixed_joint: origin xyz=-0.01061979999999986 -0.10939100000000002 0.15174599999999996 rpy=-3.1415926535897913 1.308997006967741 2.3056457336008695e-15 -> xyz=0.01160250023188351 0.14719399989874468 0.2765873999902195 rpy=0.0790794230156212 -0.052031613930206826 -0.27527862099575323
- joint l_sole_fixed_joint: origin xyz=0.007360800000000025 -0.07010000006925801 -0.6244860000000001 rpy=9.99783810877977e-9 -1.2618488420823581e-8 3.1415926509108907 -> xyz=0.048929999999999994 0.06475 -0.6325890000000001 rpy=0 -0 0
- joint l_upper_arm_fixed_joint: origin xyz=-0.025619799999999887 -0.109391 0.09499999999999996 rpy=3.1415926535897922 -1.1657341758564144e-15 -3.1415926535897927 -> xyz=0.013208121959356507 0.14858702204000246 0.2541880957564809 rpy=0.0790794230156212 -0.052031613930206826 -0.27527862099575323
- joint l_upper_leg_fixed_joint: origin xyz=0.007309000000000008 -0.07010000000000001 -0.20861299999999994 rpy=0 -0 -3.141592653589793 -> xyz=0.011049999999999997 0.05855 -0.16960000000000003 rpy=0 -0 0
- joint l_wrist_1_fixed_joint: origin xyz=-0.008469800000000067 -0.10939799999999984 -0.12656000000000006 rpy=-3.141592653589789 1.3089970069677406 4.372177745413122e-15 -> xyz=0.04547212334915017 0.1655890223793864 -0.030229004065574397 rpy=0.0790794230156212 -0.052031613930206826 -0.27527862099575323
- joint neck_1_fixed_joint: origin xyz=-0.010809299999999869 0.014299999999999986 0.254797 rpy=1.5707963267948961 -0 -1.5707963267948961 -> xyz=-0.00378849 0 0.3627695 rpy=0 -0 0
- joint neck_2_fixed_joint: origin xyz=-0.031609269999999856 1.9073497642407844e-10 0.264297 rpy=1.5707963267948961 -0 -1.5707963267948961 -> xyz=0.0048615099999999994 0 0.4117695 rpy=0 -0 0
- joint r_ankle_pitch: axis -6.661338147750938e-16 1 4.440892098500625e-16 -> 0 1 0; origin xyz=0 0 -0.20049999999999996 rpy=0 0.2617991794798451 0 -> xyz=0 5.000000000000004e-4 -0.255989 rpy=0 -0 0
- joint r_ankle_roll: axis -0.9999999999999927 -6.013653080356639e-16 1.197939310368565e-7 -> -1 0 0; origin xyz=0 0 0 rpy=0 -0 0 -> xyz=-0.052750000000000005 0.018200000000000008 -0.03500000000000003 rpy=0 -0 0
- joint r_arm_ft_sensor_fixed_joint: origin xyz=-0.025619800000000033 0.10939100000000002 0.09499999999999997 rpy=3.141592653589793 -1.1657341758564144e-15 -3.141592653589793 -> xyz=0.011602500000000036 -0.14719400000000007 0.27658740000000004 rpy=-0.07907934249382903 -0.0520316044795478 0.2752784843541201
- joint r_elbow_1_fixed_joint: origin xyz=-0.02561980000000012 0.08689110000000004 0.015739999999999976 rpy=3.141592653589792 -1.308997006967741 -3.141592653589792 -> xyz=0.031246121282148414 -0.1520930222338017 0.13144299574009638 rpy=-0.07907934249382903 -0.0520316044795478 0.2752784843541201
- joint r_forearm_fixed_joint: origin xyz=-0.010619800000000148 0.10939100000000007 -0.020060000000000036 rpy=3.141592653589792 -1.308997006967741 -3.141592653589792 -> xyz=0.021311021282148408 -0.16151002223380165 0.0757679957400964 rpy=-0.07907934249382903 -0.0520316044795478 0.2752784843541201
- joint r_hand_fixed_joint: origin xyz=-0.010619800000000209 0.08989810000000013 -0.12656000000000006 rpy=3.141592653589792 -1.308997006967741 -3.141592653589792 -> xyz=0.027649815623035374 -0.16337301732292386 -0.031644925317804405 rpy=-0.07907934249382903 -0.0520316044795478 0.2752784843541201
- joint r_hip_3_fixed_joint: origin xyz=-8.575000000000041e-4 0 -0.07429999999999995 rpy=3.141592653589793 -0 0 -> xyz=0.036699999999999997 0 -0.08969999999999995 rpy=0 -0 0
- joint r_hip_pitch: axis -2.2204460492503136e-16 -1 0 -> 0 -1 0; origin xyz=0.006451499999999992 0.025999999999999968 -0.11991299999999999 rpy=0 -0 -3.141592653589793 -> xyz=0.0216 -0.040549999999999996 0 rpy=0 -0 0
- joint r_hip_roll: axis -1 0 -2.2204460492503136e-16 -> -1 0 0; origin xyz=0 -0.04409999999999998 0 rpy=0 -0 0 -> xyz=-0.0473 -0.03310000000000001 -0.009000000000000008 rpy=0 -0 0
- joint r_hip_yaw: axis 0 -2.2204460492503136e-16 -1 -> 0 0 -1; origin xyz=-8.575000000000041e-4 -1.763491390772188e-18 -0.08869999999999995 rpy=0 -0 0 -> xyz=0.036699999999999997 0.015000000000000006 -0.16060000000000002 rpy=0 -0 0
- joint r_knee: axis -2.2204460492503136e-16 -1 0 -> 0 -1 0; origin xyz=0 0 -0.14582499999999995 rpy=0 -0 0 -> xyz=0.015000000000000003 -0.0249 -0.10619999999999996 rpy=0 -0 0
- joint r_leg_ft_sensor_fixed_joint: origin xyz=-8.575000000000041e-4 0 -0.07429999999999995 rpy=3.141592653589793 -0 0 -> xyz=0.036699999999999997 0 -0.08969999999999995 rpy=0 -0 0
- joint r_shoulder_1_fixed_joint: origin xyz=-0.01346679999999996 0.120016 0.1748 rpy=-1.5707963267948963 -3.5871833949913145e-16 2.094395210586932 -> xyz=-0.020835100000000002 -0.0397423 0.3026729 rpy=-0.25326164431680925 2.3014774394592079e-7 0.26179970938509745
- joint r_shoulder_2_fixed_joint: origin xyz=-0.021982999999999957 0.106346 0.1748 rpy=-3.141592629949768 -1.3089970275211211 -2.879793377150528 -> xyz=0.014310500000000032 -0.14197200000000007 0.33100070000000004 rpy=-0.07907934249382903 -0.0520316044795478 0.2752784843541201
- joint r_shoulder_3_fixed_joint: origin xyz=-0.010619799999999992 0.109391 0.15171199999999999 rpy=3.141592653589792 -1.308997006967741 -3.141592653589792 -> xyz=0.011602500000000036 -0.14719400000000007 0.27658740000000004 rpy=-0.07907934249382903 -0.0520316044795478 0.2752784843541201
- joint r_sole_fixed_joint: origin xyz=0.0179502979936772 -7.841709392865824e-12 -0.06719161993268341 rpy=-1.2132694871910076e-9 -0.2617991810276664 3.14017499256229e-10 -> xyz=0.07563 0 -0.06579999999999997 rpy=0 -0 0
- joint r_upper_arm_fixed_joint: origin xyz=-0.025619800000000033 0.10939100000000002 0.09499999999999997 rpy=3.141592653589793 -1.1657341758564144e-15 -3.141592653589793 -> xyz=0.013208121282148412 -0.14858702223380166 0.2541880957400964 rpy=-0.07907934249382903 -0.0520316044795478 0.2752784843541201
- joint r_wrist_1_fixed_joint: origin xyz=-0.008169800000000213 0.10939800000000013 -0.12656000000000006 rpy=3.141592653589792 -1.308997006967741 -3.141592653589792 -> xyz=0.045183921282148404 -0.16567102223380167 -0.030245004259903563 rpy=-0.07907934249382903 -0.0520316044795478 0.2752784843541201
- joint torso_1_fixed_joint: origin xyz=0 0.02693479999999999 0 rpy=1.5707963267948961 -0 -1.5707963267948961 -> xyz=0 0 0.0605 rpy=0 -0 0
- joint torso_2_fixed_joint: origin xyz=0.05734460000000004 1.9073502152688881e-10 0.03199999999999997 rpy=1.5707963267948961 -0 -1.5707963267948961 -> xyz=0 0 0.133 rpy=0 -0 0
